Commit message: update file organization

File: picknik_test_stand_description/urdf/mock_grappler.urdf.xacro (robot description, xacro)
@@ -7,5 +7,5 @@
     <!-- Constants -->
     <xacro:property name="x_origin" value="${pi/2.0}" />
-    <xacro:property name="y_origin" value="0.0" />
+    <xacro:property name="y_origin" value="${pi}" />
     <xacro:property name="z_origin" value="${pi/2.0}" />
     <!-- Description -->
