Commit message: added camera xacros to package

File: picknik_test_stand_description/urdf/materials.urdf.xacro (robot description, xacro)
@@ -2,4 +2,10 @@
 <robot xmlns:xacro="http://wiki.ros.org/xacro">
   <xacro:macro name="materials" >
+    <material name="aluminum">
+      <color rgba="0.5 0.5 0.5 1"/>
+    </material>
+    <material name="plastic">
+      <color rgba="0.1 0.1 0.1 1"/>
+    </material>
     <material name="burgandy">
       <color rgba="0.502 0.0 0.125 0.4" />

File: picknik_test_stand_description/urdf/picknik_test_stand.urdf.xacro (robot description, xacro)
@@ -3,5 +3,6 @@
 <!-- Include all macros -->
   <xacro:include filename="$(find ur_description)/urdf/inc/ur5_macro.xacro" />
-  <xacro:include filename="$(find realsense2_description)/urdf/_d415.urdf.xacro" />
+  <xacro:include filename="$(find picknik_test_stand_description)/urdf/_d415.urdf.xacro" />
+  <xacro:include filename="$(find picknik_test_stand_description)/urdf/_l515.urdf.xacro" />
   <xacro:include filename="$(find picknik_test_stand_description)/urdf/materials.urdf.xacro" />
   <xacro:include filename="$(find picknik_test_stand_description)/urdf/bench.urdf.xacro" />
@@ -69,4 +70,7 @@
     <!-- Load the calibration plate and attach to the UR5 flange -->
     <xacro:calibration_plate parent="${seg0_prefix}flange" prefix="plate_" />
+    <xacro:sensor_l515 parent="bench_base_link" use_nominal_extrinsics="true" use_mesh="true">
+      <origin xyz="-1.3 -0.09 0.38" rpy="0 0 0"/>
+    </xacro:sensor_l515>
   </xacro:if>
 </robot>
