Commit message: fixed mount joint

File: picknik_test_stand_description/urdf/calibration_plate.urdf.xacro (robot description, xacro)
@@ -9,10 +9,10 @@
     <xacro:property name="y_size" value="0.229" />
     <xacro:property name="z_size" value="0.013" />
-    <xacro:property name="x_origin" value="0.0" />
-    <xacro:property name="y_origin" value="0.0" />
+    <xacro:property name="x_origin" value="0.106" />
+    <xacro:property name="y_origin" value="-0.0745" />
     <xacro:property name="z_origin" value="0.0065" />
-    <xacro:property name="x_mount" value="0.106" />
-    <xacro:property name="y_mount" value="-0.0745" />
-    <xacro:property name="z_mount" value="0.0" />
+    <xacro:property name="r_mount" value="0.0" />
+    <xacro:property name="p_mount" value="${pi/2}" />
+    <xacro:property name="y_mount" value="0.0" />
     <link name="${prefix}base_link" >
       <visual>
@@ -33,5 +33,5 @@
       <parent link="${parent}" />
       <child link="${prefix}base_link" />
-      <origin xyz="${x_mount} ${y_mount} ${z_mount}" rpy="0.0 0.0 0.0" />
+      <origin xyz="0.0 0.0 0.0" rpy="${r_mount} ${p_mount} ${y_mount}" />
     </joint>
   </xacro:macro>

Commit message: updated plate position

File: picknik_test_stand_description/urdf/calibration_plate.urdf.xacro (robot description, xacro)
@@ -12,7 +12,7 @@
     <xacro:property name="y_origin" value="-0.0745" />
     <xacro:property name="z_origin" value="0.0065" />
-    <xacro:property name="r_mount" value="0.0" />
-    <xacro:property name="p_mount" value="${pi/2}" />
-    <xacro:property name="y_mount" value="0.0" />
+    <xacro:property name="r_mount" value="${pi/2}" />
+    <xacro:property name="p_mount" value="0.0" />
+    <xacro:property name="y_mount" value="${pi/2}" />
     <link name="${prefix}base_link" >
       <visual>
