Commit message: updated for new room and for arm prefix

File: picknik_test_stand_description/urdf/bench.urdf.xacro (robot description, xacro)
@@ -9,7 +9,7 @@
     <xacro:property name="y_size" value="0.62" />
     <xacro:property name="z_size" value="0.92" />
-    <xacro:property name="x_origin" value="-0.465" />
-    <xacro:property name="y_origin" value="-0.175" />
-    <xacro:property name="z_origin" value="0.46" />
+    <xacro:property name="x_origin" value="${x_size / 2}" />
+    <xacro:property name="y_origin" value="${y_size / 2}" />
+    <xacro:property name="z_origin" value="-${z_size / 2}" />
     <!-- Description -->
     <link name="${prefix}base_link" >
@@ -31,5 +31,5 @@
       <parent link="${parent}" />
       <child link="${prefix}base_link" />
-      <origin xyz="0.0 0.0 0.0" rpy="0.0 0.0 0.0" />
+      <origin xyz="0.0 0.0 ${z_size}" rpy="0.0 0.0 0.0" />
     </joint>
   </xacro:macro>

File: picknik_test_stand_description/urdf/materials.urdf.xacro (robot description, xacro)
@@ -17,4 +17,7 @@
         <color rgba="0.3 0.3 0.3 0.8" />
     </material>
+    <material name="light_grey">
+        <color rgba="0.2 0.2 0.2 0.4" />
+    </material>
     <material name="silver">
       <color rgba="0.75 0.75 0.75 1.0" />
