Commit message: switch to standard joint names to easily work with the controller

File: picknik_test_stand_description/config/picknik_test_stand.srdf.xacro (robot description, xacro)
@@ -10,5 +10,5 @@
     <!--CHAINS: When a chain is specified, all the links along the chain (including endpoints) are included in the group. Additionally, all the joints that are parents to included links are also included. This means that joints along the chain and the parent joint of the base link are included in the group-->
     <!--SUBGROUPS: Groups can also be formed by referencing to already defined group names-->
-    <xacro:property name="ur5_prefix" value="seg0_" />
+    <xacro:property name="ur5_prefix" value="" />
     <group name="manipulator">
         <chain base_link="${ur5_prefix}base_link" tip_link="${ur5_prefix}wrist_3_link" />

File: picknik_test_stand_description/urdf/picknik_test_stand.urdf.xacro (robot description, xacro)
@@ -14,5 +14,5 @@
   <xacro:property name="camera_calibration_file" value="$(find picknik_test_stand_description)/config/camera_calibration.yaml" />
   <xacro:property name="camera_calibration" value="${load_yaml(camera_calibration_file)}" />
-  <xacro:property name="seg0_prefix" value="seg0_" />
+  <xacro:property name="seg0_prefix" value="" />
 <!-- Parameters -->
   <xacro:arg name="joint_limit_params" default=""/>

Commit message: added ability to change end effector

File: picknik_test_stand_description/config/picknik_test_stand.srdf.xacro (robot description, xacro)
@@ -50,7 +50,8 @@
     <disable_collisions link1="${ur5_prefix}wrist_1_link" link2="${ur5_prefix}wrist_3_link" reason="Never" />
     <disable_collisions link1="${ur5_prefix}wrist_2_link" link2="${ur5_prefix}wrist_3_link" reason="Adjacent" />
-    <disable_collisions link1="${ur5_prefix}wrist_3_link" link2="grappler_base_link" reason="Adjacent" />
     <disable_collisions link1="${ur5_prefix}base_link_inertia" link2="bench_base_link" reason="Adjacent" />
     <disable_collisions link1="bench_base_link" link2="wall_base_link" reason="Adjacent" />
+    <disable_collisions link1="${ur5_prefix}wrist_3_link" link2="grappler_base_link" reason="Adjacent" />
     <disable_collisions link1="grappler_base_link" link2="camera_link" reason="Adjacent" />
+    <disable_collisions link1="${ur5_prefix}wrist_3_link" link2="plate_base_link" reason="Adjacent" />
 </robot>

File: picknik_test_stand_description/urdf/materials.urdf.xacro (robot description, xacro)
@@ -2,9 +2,12 @@
 <robot xmlns:xacro="http://wiki.ros.org/xacro">
   <xacro:macro name="materials" >
+    <material name="burgandy">
+      <color rgba="0.502 0.0 0.125 0.4" />
+    </material>
+    <material name="brown">
+      <color rgba="0.55 0.35 0.17 1" />
+    </material>
     <material name="grey">
         <color rgba="0.3 0.3 0.3 0.8" />
-    </material>
-    <material name="burgandy">
-      <color rgba="0.502 0.0 0.125 0.4" />
     </material>
     <material name="silver">

File: picknik_test_stand_description/urdf/picknik_test_stand.urdf.xacro (robot description, xacro)
@@ -8,7 +8,6 @@
   <xacro:include filename="$(find picknik_test_stand_description)/urdf/wall.urdf.xacro" />
   <xacro:include filename="$(find picknik_test_stand_description)/urdf/mock_grappler.urdf.xacro" />
+  <xacro:include filename="$(find picknik_test_stand_description)/urdf/calibration_plate.urdf.xacro" />
 <!-- Constants -->
-  <xacro:property name="yaml_file" value="$(find picknik_test_stand/config/picknik_test_stand.yaml" />
-  <xacro:property name="properties" value="${load_yaml(yaml_file)}" />
   <xacro:property name="arm_height" value="0.92" />
   <xacro:property name="camera_calibration_file" value="$(find picknik_test_stand_description)/config/camera_calibration.yaml" />
@@ -29,8 +28,11 @@
   <xacro:arg name="safety_pos_margin" default="0.15"/>
   <xacro:arg name="safety_k_position" default="20"/>
+  <xacro:arg name="end_effector" default="none" />
+  <!-- Note: converting this to property so if statement can be used later, not sure of a better way to do this -->
+  <xacro:property name="end_effector" value="$(arg end_effector)" />
 <!-- Build the scence -->
   <!-- Common materials -->
   <xacro:materials />
-  <!-- Create the base link at the orgin of the scene -->
+  <!-- Create the simulated base link at the orgin of the scene -->
   <link name="tractor_base" />
   <!-- Load the work bench and attach to the base link -->
@@ -55,9 +57,16 @@
     <origin xyz="0.0 0.0 ${arm_height}" rpy="0.0 0.0 0.0" />
   </joint>
-  <!-- Load the mock grappler and attach to the UR5 flange -->
-  <xacro:mock_grappler parent="${seg0_prefix}flange" prefix="grappler_" />
-  <!-- Load a D415 RealSense camera and attach to mock grappler -->
-  <xacro:sensor_d415 parent="grappler_base_link" use_nominal_extrinsics="true" use_mesh="true">
-    <origin xyz="${camera_calibration['arm_camera']['xyz']}" rpy="${camera_calibration['arm_camera']['rpy']}" />
-  </xacro:sensor_d415>
+  <!-- Load the selected end effector -->
+  <xacro:if value="${end_effector == 'mock_grappler'}" >
+    <!-- Load the mock grappler and attach to the UR5 flange -->
+    <xacro:mock_grappler parent="${seg0_prefix}flange" prefix="grappler_" />
+    <!-- Load a D415 RealSense camera and attach to mock grappler -->
+    <xacro:sensor_d415 parent="grappler_base_link" use_nominal_extrinsics="true" use_mesh="true">
+      <origin xyz="${camera_calibration['arm_camera']['xyz']}" rpy="${camera_calibration['arm_camera']['rpy']}" />
+    </xacro:sensor_d415>
+  </xacro:if>
+  <xacro:if value="${end_effector == 'calibration_plate'}" >
+    <!-- Load the calibration plate and attach to the UR5 flange -->
+    <xacro:calibration_plate parent="${seg0_prefix}flange" prefix="plate_" />
+  </xacro:if>
 </robot>

Commit message: added parameter to semantic description

File: picknik_test_stand_description/config/picknik_test_stand.srdf.xacro (robot description, xacro)
@@ -10,5 +10,10 @@
     <!--CHAINS: When a chain is specified, all the links along the chain (including endpoints) are included in the group. Additionally, all the joints that are parents to included links are also included. This means that joints along the chain and the parent joint of the base link are included in the group-->
     <!--SUBGROUPS: Groups can also be formed by referencing to already defined group names-->
+<!-- PARAMETERS -->
     <xacro:property name="ur5_prefix" value="" />
+    <xacro:arg name="end_effector" default="none"/>
+    <!-- Note: converting this to property so if statement can be used later, not sure of a better way to do this -->
+    <xacro:property name="end_effector" value="$(arg end_effector)" />
+<!-- GROUP DEFINITIONS -->
     <group name="manipulator">
         <chain base_link="${ur5_prefix}base_link" tip_link="${ur5_prefix}wrist_3_link" />
@@ -17,5 +22,5 @@
         <link name="tool0" />
     </group> -->
-    <!--GROUP STATES: Purpose: Define a named state for a particular group, in terms of joint values. This is useful to define states like 'folded arms'-->
+<!--GROUP STATES: Purpose: Define a named state for a particular group, in terms of joint values. This is useful to define states like 'folded arms'-->
     <group_state name="home" group="manipulator">
         <joint name="${ur5_prefix}elbow_joint" value="0" />
@@ -34,9 +39,9 @@
         <joint name="${ur5_prefix}wrist_3_joint" value="0" />
     </group_state>
-    <!--END EFFECTOR: Purpose: Represent information about an end effector.-->
+<!--END EFFECTOR: Purpose: Represent information about an end effector.-->
     <!-- <end_effector name="moveit_ee" parent_link="tool0" group="endeffector" /> -->
-    <!--VIRTUAL JOINT: Purpose: this element defines a virtual joint between a robot link and an external frame of reference (considered fixed with respect to the robot)-->
+<!--VIRTUAL JOINT: Purpose: this element defines a virtual joint between a robot link and an external frame of reference (considered fixed with respect to the robot)-->
     <virtual_joint name="fixed_base" type="fixed" parent_frame="world" child_link="tractor_base" />
-    <!--DISABLE COLLISIONS: By default it is assumed that any link of the robot could potentially come into collision with any other link in the robot. This tag disables collision checking between a specified pair of links. -->
+<!--DISABLE COLLISIONS: By default it is assumed that any link of the robot could potentially come into collision with any other link in the robot. This tag disables collision checking between a specified pair of links. -->
     <disable_collisions link1="${ur5_prefix}base_link_inertia" link2="${ur5_prefix}shoulder_link" reason="Adjacent" />
     <disable_collisions link1="${ur5_prefix}base_link_inertia" link2="${ur5_prefix}upper_arm_link" reason="Never" />
@@ -52,6 +57,12 @@
     <disable_collisions link1="${ur5_prefix}base_link_inertia" link2="bench_base_link" reason="Adjacent" />
     <disable_collisions link1="bench_base_link" link2="wall_base_link" reason="Adjacent" />
-    <disable_collisions link1="${ur5_prefix}wrist_3_link" link2="grappler_base_link" reason="Adjacent" />
-    <disable_collisions link1="grappler_base_link" link2="camera_link" reason="Adjacent" />
-    <disable_collisions link1="${ur5_prefix}wrist_3_link" link2="plate_base_link" reason="Adjacent" />
+    <!-- Mock grappler -->
+    <xacro:if value="${end_effector == 'mock_grappler'}" >
+        <disable_collisions link1="${ur5_prefix}wrist_3_link" link2="grappler_base_link" reason="Adjacent" />
+        <disable_collisions link1="grappler_base_link" link2="camera_link" reason="Adjacent" />
+    </xacro:if>
+    <!-- Calibration plate -->
+    <xacro:if value="${end_effector == 'calibration_plate'}" >
+        <disable_collisions link1="${ur5_prefix}wrist_3_link" link2="plate_base_link" reason="Adjacent" />
+    </xacro:if>
 </robot>
