Commit message: updated for new room and for arm prefix

File: picknik_test_stand_description/config/picknik_test_stand.srdf.xacro (robot description, xacro)
@@ -13,5 +13,5 @@
     <xacro:include filename="$(find picknik_test_stand_description)/config/calibration_positions.srdf.xacro" />
 <!-- PARAMETERS -->
-    <xacro:property name="ur5_prefix" value="" />
+    <xacro:property name="ur5_prefix" value="ur5_" />
     <xacro:arg name="end_effector" default="none"/>
     <!-- Note: converting this to property so if statement can be used later, not sure of a better way to do this -->
@@ -44,5 +44,5 @@
     <!-- <end_effector name="moveit_ee" parent_link="tool0" group="endeffector" /> -->
 <!--VIRTUAL JOINT: Purpose: this element defines a virtual joint between a robot link and an external frame of reference (considered fixed with respect to the robot)-->
-    <virtual_joint name="fixed_base" type="fixed" parent_frame="world" child_link="tractor_base" />
+    <virtual_joint name="fixed_base" type="fixed" parent_frame="world" child_link="base_link" />
 <!--DISABLE COLLISIONS: By default it is assumed that any link of the robot could potentially come into collision with any other link in the robot. This tag disables collision checking between a specified pair of links. -->
     <disable_collisions link1="${ur5_prefix}base_link_inertia" link2="${ur5_prefix}shoulder_link" reason="Adjacent" />
@@ -58,7 +58,10 @@
     <disable_collisions link1="${ur5_prefix}wrist_2_link" link2="${ur5_prefix}wrist_3_link" reason="Adjacent" />
     <disable_collisions link1="${ur5_prefix}base_link_inertia" link2="bench_base_link" reason="Adjacent" />
-    <disable_collisions link1="bench_base_link" link2="wall0_base_link" reason="Adjacent" />
-    <disable_collisions link1="bench_base_link" link2="wall1_base_link" reason="Adjacent" />
-    <disable_collisions link1="wall0_base_link" link2="wall1_base_link" reason="Adjacent" />
+    <disable_collisions link1="bench_base_link" link2="west_wall_base_link" reason="Never" />
+    <disable_collisions link1="bench_base_link" link2="safety_wall_base_link" reason="Never" />
+    <disable_collisions link1="bench_base_link" link2="safety_wall_base_link" reason="Never" />
+    <disable_collisions link1="west_wall_base_link" link2="north_wall_base_link" reason="Adjacent" />
+    <disable_collisions link1="west_wall_base_link" link2="safety_wall_base_link" reason="Adjacent" />
+    <disable_collisions link1="north_wall_base_link" link2="safety_wall_base_link" reason="Never" />
     <!-- Mock grappler -->
     <xacro:if value="${end_effector == 'mock_grappler'}" >
@@ -69,5 +72,5 @@
     <xacro:if value="${end_effector == 'calibration_plate'}" >
         <disable_collisions link1="${ur5_prefix}wrist_3_link" link2="plate_base_link" reason="Adjacent" />
-        <xacro:calibration_positions />
+        <xacro:calibration_positions prefix="${ur5_prefix}"/>
     </xacro:if>
 </robot>

File: picknik_test_stand_description/urdf/picknik_test_stand.urdf.xacro (robot description, xacro)
@@ -11,8 +11,21 @@
   <xacro:include filename="$(find picknik_test_stand_description)/urdf/calibration_plate.urdf.xacro" />
 <!-- Constants -->
-  <xacro:property name="arm_height" value="0.92" />
+  <xacro:property name="arm_mounting_position" value="1.05 .495 0.0" />
+  <xacro:property name="arm_mounting_orientation" value="0.0 0.0 0.0" />
+  <xacro:property name="west_wall_mounting_position" value="-0.184 -0.2 0.0" />
+  <xacro:property name="west_wall_mounting_orientation" value="0.0 0.0 3.1416" />
+  <xacro:property name="west_wall_width" value="4.5" />
+  <xacro:property name="west_wall_color" value="light_grey" />
+  <xacro:property name="north_wall_mounting_position" value="-0.184 -0.20 0.0" />
+  <xacro:property name="north_wall_mounting_orientation" value="0.0 0.0 -1.5708" />
+  <xacro:property name="north_wall_width" value="2.4" />
+  <xacro:property name="north_wall_color" value="light_grey" />
+  <xacro:property name="safety_wall_mounting_position" value="1.7 -0.20 0.0" />
+  <xacro:property name="safety_wall_mounting_orientation" value="0.0 0.0 -1.5708" />
+  <xacro:property name="safety_wall_width" value="2.4" />
+  <xacro:property name="safety_wall_color" value="burgandy" />
   <xacro:property name="camera_calibration_file" value="$(find picknik_test_stand_description)/config/camera_calibration.yaml" />
   <xacro:property name="camera_calibration" value="${load_yaml(camera_calibration_file)}" />
-  <xacro:property name="seg0_prefix" value="" />
+  <xacro:property name="arm_prefix" value="ur5_" />
 <!-- Parameters -->
   <xacro:arg name="joint_limit_params" default=""/>
@@ -36,13 +49,32 @@
   <xacro:materials />
   <!-- Create the simulated base link at the orgin of the scene -->
-  <link name="tractor_base" />
+  <link name="base_link" />
   <!-- Load the work bench and attach to the base link -->
-  <xacro:bench parent="tractor_base" prefix="bench_" />
+  <xacro:bench parent="base_link" prefix="bench_" />
   <!-- Load the imaginary safety wall and attach to the work bench -->
-  <xacro:wall parent="bench_base_link" prefix="wall0_" mount_xyz="0.0 -0.51 0.0" mount_rpy="-1.5708 0.0 0.0"/>
-  <xacro:wall parent="bench_base_link" prefix="wall1_" mount_xyz="0.5 0.0 0.0" mount_rpy="-1.5708 0.0 -1.5708"/>
+  <xacro:wall parent="base_link" prefix="west_wall_"
+    width="${west_wall_width}"
+    dir="1"
+    mount_xyz="${west_wall_mounting_position}"
+    mount_rpy="${west_wall_mounting_orientation}"
+    color="${west_wall_color}"
+    />
+  <xacro:wall parent="base_link" prefix="north_wall_"
+    width="${north_wall_width}"
+    dir="-1"
+    mount_xyz="${north_wall_mounting_position}"
+    mount_rpy="${north_wall_mounting_orientation}"
+    color="${north_wall_color}"
+    />
+  <xacro:wall parent="base_link" prefix="safety_wall_"
+    width="${safety_wall_width}"
+    dir="1"
+    mount_xyz="${safety_wall_mounting_position}"
+    mount_rpy="${safety_wall_mounting_orientation}"
+    color="${safety_wall_color}"
+    />
   <!-- Load the UR5 -->
   <xacro:ur5_robot
-    prefix="${seg0_prefix}"
+    prefix="${arm_prefix}"
     joint_limits_parameters_file="$(arg joint_limit_params)"
     kinematics_parameters_file="$(arg kinematics_params)"
@@ -56,11 +88,11 @@
   <joint name="bench_to_ur5_robot" type="fixed" >
     <parent link="bench_base_link" />
-    <child link="${seg0_prefix}base_link" />
-    <origin xyz="0.0 0.0 ${arm_height}" rpy="0.0 0.0 0.0" />
+    <child link="${arm_prefix}base_link" />
+    <origin xyz="${arm_mounting_position}" rpy="${arm_mounting_orientation}" />
   </joint>
   <!-- Load the selected end effector -->
   <xacro:if value="${end_effector == 'mock_grappler'}" >
     <!-- Load the mock grappler and attach to the UR5 flange -->
-    <xacro:mock_grappler parent="${seg0_prefix}flange" prefix="grappler_" />
+    <xacro:mock_grappler parent="${arm_prefix}flange" prefix="grappler_" />
     <!-- Load a D415 RealSense camera and attach to mock grappler -->
     <xacro:sensor_d415 parent="grappler_base_link" use_nominal_extrinsics="true" use_mesh="true">
@@ -70,6 +102,6 @@
   <xacro:if value="${end_effector == 'calibration_plate'}" >
     <!-- Load the calibration plate and attach to the UR5 flange -->
-    <xacro:calibration_plate parent="${seg0_prefix}flange" prefix="plate_" />
-    <xacro:sensor_l515 parent="bench_base_link" use_nominal_extrinsics="true" use_mesh="true">
+    <xacro:calibration_plate parent="${arm_prefix}flange" prefix="plate_" />
+    <xacro:sensor_l515 parent="base_link" use_nominal_extrinsics="true" use_mesh="true">
       <origin xyz="${camera_calibration['calibration_camera']['xyz']}" rpy="${camera_calibration['calibration_camera']['rpy']}"/>
     </xacro:sensor_l515>

File: picknik_test_stand_description/urdf/wall.urdf.xacro (robot description, xacro)
@@ -4,14 +4,18 @@
       prefix
       parent
+      width
+      dir
       mount_xyz
-      mount_rpy"
+      mount_rpy
+      color"
   >
     <!-- Constants -->
-    <xacro:property name="x_size" value="2.0" />
-    <xacro:property name="y_size" value="2.5" />
-    <xacro:property name="z_size" value="0.025" />
-    <xacro:property name="x_origin" value="0.0" />
-    <xacro:property name="y_origin" value="-1.25" />
-    <xacro:property name="z_origin" value="0.0125" />
+    <xacro:property name="flip" value="${dir}" />
+    <xacro:property name="x_size" value="${width}" />
+    <xacro:property name="y_size" value="0.025" />
+    <xacro:property name="z_size" value="2.5" />
+    <xacro:property name="x_origin" value="-${x_size / 2}" />
+    <xacro:property name="y_origin" value="${dir * y_size / 2}" />
+    <xacro:property name="z_origin" value="${z_size / 2}" />
     <link name="${prefix}base_link" >
       <visual>
@@ -20,5 +24,5 @@
         </geometry>
         <origin xyz="${x_origin} ${y_origin} ${z_origin}" rpy="0.0 0.0 0.0" />
-        <material name="burgandy" />
+        <material name="${color}" />
       </visual>
       <collision>
